File: pcb/macropad.kicad_pcb (KiCad board)
At the start: 2 copper layers, 135 x 79.3 mm, 36 parts, among them J1 Conn_01x02_Pin, SW1 SW_Push, SW10 SW_Push, SW11 SW_Push, SW12 SW_Push, SW13 SW_Push, SW14 SW_Push, SW15 SW_Push, SW16 SW_Push, SW17 SW_DIP_x01, SW18 SW_Push, SW2 SW_Push, SW3 SW_Push, SW4 SW_Push, SW5 SW_Push, SW6 SW_Push, SW7 SW_Push, SW8 SW_Push, SW9 SW_Push, U2 ProMicro

Commit message: More laying out
Parts:
- D1, D10, D11, D12, D13, D14, D15, D16, D2, D3, D4, D5, D6, D7, D8, D9: footprint Diode_SMD:D_0201_0603Metric -> Diode_SMD:D_SOD-323
- J1: footprint Connector_PinHeader_2.54mm:PinHeader_1x02_P2.54mm_Horizontal -> Connector_PinHeader_2.54mm:PinHeader_1x02_P2.54mm_Vertical
- SW1, SW10, SW11, SW12, SW13, SW14, SW15, SW16, SW2, SW3, SW4, SW5, SW6, SW7, SW8, SW9: footprint key-switches:SW_MX_LowProfile_Kailh_Choc_V1V2_THT_Hybrid -> key-switches:SW_MX_Kailh_Choc_V1V2_HotSwap_Hybrid
- SW17: footprint Button_Switch_SMD:SW_SPST_REED_CT10-XXXX-G1 -> Button_Switch_SMD:SW_SPDT_Shouhan_MSK12C02; moved to B.Cu
- SW18: footprint Button_Switch_THT:SW_PUSH_6mm -> Button_Switch_SMD:SW_SPST_EVQP2_MiddlePushTravel_H2.5mm; moved to B.Cu
- U2: footprint TheOneProMicro:TheOneProMicro -> TheOneProMicro:TheOneProMacro
- moved SW17 117.3 mm to (52.7, 28.0)
- moved SW18 114.4 mm to (47.7, 48.0), turned to 90 degrees
- moved J1 101.6 mm to (67.1, 27.9), turned to 90 degrees
- moved U2 88.8 mm to (37.0, 43.1)
Connections:
- SW17 pad 2: Net-(J1-Pin_1) -> Net-(J1-Pin_2)
- SW18 pad 2: Net-(SW18-Pad2) -> Net-(J1-Pin_1)
- U2 pad 13: unconnected-(U2-GP21-Pad13) -> COL1
- U2 pad 14: unconnected-(U2-GP23-Pad14) -> COL0
- U2 pad 30: unconnected-(U2-GP16-Pad30) -> COL3
- U2 pad 33: Net-(J1-Pin_2) -> Net-(J1-Pin_1)
- U2 pad 8: COL1 -> COL2
Routing:
- net ROW0: track 0.00 -> 77.9 mm
- net COL1: track 0.00 -> 73.4 mm, vias 0 -> 4
- net COL0: track 0.00 -> 72.0 mm, vias 0 -> 4
- net COL2: track 0.00 -> 72.0 mm, vias 0 -> 4
- net COL3: track 0.00 -> 72.0 mm, vias 0 -> 4
- net ROW2: track 0.00 -> 66.0 mm
- net ROW1: track 0.00 -> 61.3 mm
- net ROW3: track 0.00 -> 61.3 mm
- net Net-(U2-RST): track 0.00 -> 40.3 mm, vias 0 -> 1
- net Net-(J1-Pin_1): track 16.4 -> 48.8 mm, vias 0 -> 1
- net Net-(U2-GP11(B+)): track 0.00 -> 23.2 mm
- net Net-(D10-A): track 1.19 -> 22.3 mm
- net Net-(D3-A): track 1.19 -> 22.3 mm
- net Net-(D4-A): track 1.19 -> 22.1 mm
- net Net-(D2-A): track 1.19 -> 22.1 mm
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Other:
- board size 135 x 79.3 mm -> 81.3 x 81.3 mm
- board text added: "GP11/B+"

Commit message: More laying out
Connections:
- U2 pad 14: COL0 -> ROW2
- U2 pad 16: ROW2 -> COL0
Routing:
- net COL3: track 72.0 -> 148.9 mm, vias 4 -> 5
- net ROW3: track 61.3 -> 125.7 mm, vias 0 -> 1
- net COL2: track 72.0 -> 113.3 mm
- net COL1: track 73.4 -> 111.4 mm, vias 4 -> 6
- net ROW2: track 66.0 -> 101.7 mm, vias 0 -> 2
- net ROW1: track 61.3 -> 86.8 mm
- net Net-(D5-A): track 6.81 -> 23.5 mm
- net COL0: track 72.0 -> 88.2 mm
- net Net-(D9-A): track 6.81 -> 22.3 mm
Other:
- board text added: "+"
- board text added: "-"
- board text added: "THIS SIDE UP"

Commit message: More laying out
Parts:
- removed SW18: SW_Push, Button_Switch_SMD:SW_SPST_EVQP2_MiddlePushTravel_H2.5mm
- added RESET: SW_Push, Button_Switch_SMD:SW_SPST_TS-1088-xR020, B.Cu at (47.6, 47.8)
- renumbered SW17 to ON/OFF
Routing:
- net Net-(U2-RST): track 40.3 -> 0.00 mm, vias 1 -> 0
- net Net-(J1-Pin_1): track 48.8 -> 24.6 mm, vias 1 -> 0
Other:
- board text added: "BATT"

Commit message: More laying out
Routing:
- net Net-(U2-RST): track 0.00 -> 32.9 mm, vias 0 -> 1
- net Net-(J1-Pin_1): track 24.6 -> 49.1 mm, vias 0 -> 1
Changed lines of the file:
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@@
 	)
 	(gr_text "-"
-		(at 63.5 28.702 0)
+		(at 65.659 28.702 0)
 		(layer "B.SilkS")
 		(effects
@@
 				(bold yes)
 			)
-			(justify left bottom)
+			(justify left bottom mirror)
 		)
 	)
 	(gr_text "+"
-		(at 70.866 28.702 0)
+		(at 73.025 28.702 0)
 		(layer "B.SilkS")
 		(effects
@@
 				(bold yes)
 			)
-			(justify left bottom)
+			(justify left bottom mirror)
 		)
 	)
@@
 		(layer "B.Cu")
 		(net 20)
+	)
+	(segment
+		(start 47.625 50.038)
+		(end 48.276 49.387)
+		(width 0.2)
+		(layer "F.Cu")
+		(net 21)
+	)
+	(segment
+		(start 48.276 49.387)
+		(end 48.276 32.782)
+		(width 0.2)
+		(layer "F.Cu")
+		(net 21)
+	)
+	(segment
+		(start 48.276 32.782)
+		(end 43.307 27.813)
+		(width 0.2)
+		(layer "F.Cu")
+		(net 21)
+	)
+	(via
+		(at 47.625 50.038)
+		(size 0.7)
+		(drill 0.3)
+		(layers "F.Cu" "B.Cu")
+		(net 21)
 	)
 	(segment
@@
 		(net 27)
 	)
+	(segment
+		(start 42.739984 31.139)
+		(end 32.361 31.139)
+		(width 0.2)
+		(layer "F.Cu")
+		(net 28)
+	)
+	(segment
+		(start 32.361 31.139)
+		(end 28.067 35.433)
+		(width 0.2)
+		(layer "F.Cu")
+		(net 28)
+	)
+	(segment
+		(start 47.625 36.024016)
+		(end 42.739984 31.139)
+		(width 0.2)
+		(layer "F.Cu")
+		(net 28)
+	)
+	(segment
+		(start 47.625 45.593)
+		(end 47.625 36.024016)
+		(width 0.2)
+		(layer "F.Cu")
+		(net 28)
+	)
+	(via
+		(at 47.625 45.593)
+		(size 0.7)
+		(drill 0.3)
+		(layers "F.Cu" "B.Cu")
+		(net 28)
+	)
+	(segment
+		(start 47.625 45.588)
+		(end 47.625 45.593)
+		(width 0.2)
+		(layer "B.Cu")
+		(net 28)
+	)
 	(embedded_fonts no)

Commit message: Improvements
Parts:
- removed ON/OFF: SW_DIP_x01, Button_Switch_SMD:SW_SPDT_Shouhan_MSK12C02
- removed RESET: SW_Push, Button_Switch_SMD:SW_SPST_TS-1088-xR020
- added SW17: SW_DIP_x01, Button_Switch_SMD:SW_SPDT_Shouhan_MSK12C02, B.Cu at (52.7, 28.0)
- added SW18: SW_Push, Button_Switch_SMD:SW_SPST_TS-1088-xR020, B.Cu at (47.6, 47.8)
Connections:
- J1 pad 2: Net-(J1-Pin_2) -> GND
- U2 pad 33: Net-(J1-Pin_1) -> GND
Routing:
- net GND: track 0.00 -> 51.3 mm, vias 0 -> 1
- net Net-(J1-Pin_1): track 49.1 -> 14.5 mm, vias 1 -> 0
- net Net-(J1-Pin_2): track 17.9 -> 0.00 mm
- net Net-(U2-RST): track 32.9 -> 30.3 mm
Other:
- board text added: "ON/OFF"
- board text added: "RESET"
