File: pcb/macropad.kicad_pcb (KiCad board)
At the start: 2 copper layers, 81.3 x 81.3 mm, 36 parts, among them J1 Conn_01x02_Pin, SW1 SW_Push, SW10 SW_Push, SW11 SW_Push, SW12 SW_Push, SW13 SW_Push, SW14 SW_Push, SW15 SW_Push, SW16 SW_Push, SW17 SW_DIP_x01, SW18 SW_Push, SW2 SW_Push, SW3 SW_Push, SW4 SW_Push, SW5 SW_Push, SW6 SW_Push, SW7 SW_Push, SW8 SW_Push, SW9 SW_Push, U2 ProMicro

Commit message: Change silkscreen text from ON/OFF to OFF - ON
Other:
- board text added: "OFF - ON"
- board text removed: "ON/OFF"
Changed lines of the file:
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@@
 		)
 	)
-	(gr_text "ON/OFF"
+	(gr_text "OFF - ON"
 		(at 52.705 32.258 0)
 		(layer "B.SilkS")
