File: pcb/macropad.kicad_sch (KiCad schematic)
At the start: 36 parts, among them J1 Conn_01x02_Pin, SW1 SW_Push, SW10 SW_Push, SW11 SW_Push, SW12 SW_Push, SW13 SW_Push, SW14 SW_Push, SW15 SW_Push, SW16 SW_Push, SW17 SW_DIP_x01, SW18 SW_Push, SW2 SW_Push, SW3 SW_Push, SW4 SW_Push, SW5 SW_Push, SW6 SW_Push, SW7 SW_Push, SW8 SW_Push, SW9 SW_Push, U2 ProMicro

Commit message: More laying out
Parts:
- D1, D10, D11, D12, D13, D14, D15, D16, D2, D3, D4, D5, D6, D7, D8, D9: footprint Diode_SMD:D_0201_0603Metric -> Diode_SMD:D_SOD-323; LCSC (none) -> C2128
- J1: footprint Connector_PinHeader_2.54mm:PinHeader_1x02_P2.54mm_Horizontal -> Connector_PinHeader_2.54mm:PinHeader_1x02_P2.54mm_Vertical
- SW1, SW10, SW11, SW12, SW13, SW14, SW15, SW16, SW2, SW3, SW4, SW5, SW6, SW7, SW8, SW9: footprint key-switches:SW_MX_LowProfile_Kailh_Choc_V1V2_THT_Hybrid -> key-switches:SW_MX_Kailh_Choc_V1V2_HotSwap_Hybrid
- SW17: footprint Button_Switch_SMD:SW_SPST_REED_CT10-XXXX-G1 -> Button_Switch_SMD:SW_SPDT_Shouhan_MSK12C02
- SW18: footprint Button_Switch_THT:SW_PUSH_6mm -> Button_Switch_SMD:SW_SPST_EVQP2_MiddlePushTravel_H2.5mm
- U2: footprint TheOneProMicro:TheOneProMicro -> TheOneProMicro:TheOneProMacro
Connections:
- net COL0: now also U2.14 (GP23); no longer U2.7 (GP4)
- net COL1: now also U2.13 (GP21); no longer U2.8 (GP5)
- net COL2: now also U2.8 (GP5); no longer U2.9 (GP6)
- net COL3: now also U2.30 (GP16); no longer U2.10 (GP7)
- net at SW17.2: now also J1.2 (Pin_2); no longer J1.1 (Pin_1)
- net at U2.33 (GP10(B-)): now also J1.1 (Pin_1), SW18.2; no longer J1.2 (Pin_2)
- net at U2.23 (GND): no longer SW18.2
- no-connect marks 23 -> 24
Other:
- moved on the sheet: D1, J1, SW1, SW10, SW11, SW12, SW13, SW14, SW15, SW16, SW17, SW18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

Commit message: More laying out
Connections:
- net COL0: now also U2.16 (GP22); no longer U2.14 (GP23)
- net ROW2: now also U2.14 (GP23); no longer U2.16 (GP22)
Changed lines of the file:
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@@
 		)
 	)
-	(global_label "ROW2"
+	(global_label "COL0"
 		(shape input)
 		(at 167.64 72.39 0)
@@
 		)
 		(property "Intersheetrefs" "${INTERSHEET_REFS}"
-			(at 175.8866 72.39 0)
+			(at 175.4633 72.39 0)
 			(effects
 				(font
@@
 		)
 	)
-	(global_label "COL0"
+	(global_label "ROW2"
 		(shape input)
 		(at 167.64 77.47 0)
@@
 		)
 		(property "Intersheetrefs" "${INTERSHEET_REFS}"
-			(at 175.4633 77.47 0)
+			(at 175.8866 77.47 0)
 			(effects
 				(font

Commit message: More laying out
Parts:
- SW18: footprint Button_Switch_SMD:SW_SPST_EVQP2_MiddlePushTravel_H2.5mm -> Button_Switch_SMD:SW_SPST_TS-1088-xR020; LCSC (none) -> C720477
Changed lines of the file:
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@@
 			)
 		)
-		(property "Footprint" "Button_Switch_SMD:SW_SPST_EVQP2_MiddlePushTravel_H2.5mm"
+		(property "Footprint" "Button_Switch_SMD:SW_SPST_TS-1088-xR020"
 			(at 171.45 52.07 0)
 			(effects
@@
 			)
 		)
+		(property "LCSC" "C720477"
+			(at 171.45 57.15 0)
+			(effects
+				(font
+					(size 1.27 1.27)
+				)
+				(hide yes)
+			)
+		)

Commit message: Improvements
Connections:
- net at SW17.2: now also J1.1 (Pin_1); no longer J1.2 (Pin_2)
- net GND: now reaches SW18.2, U2.33 (GP10(B-))
- net GND: now also J1.2 (Pin_2); no longer J1.1 (Pin_1)
Other:
- moved on the sheet: J1
Changed lines of the file:
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@@
+	)
+	(junction
+		(at 130.81 45.72)
+		(diameter 0)
+		(color 0 0 0 0)
 	)
 	(junction
@@
 	)
 	(junction
-		(at 179.07 48.26)
-		(diameter 0)
-		(color 0 0 0 0)
-	)
-	(junction
 		(at 93.98 50.8)
 		(diameter 0)
@@
 	(wire
 		(pts
+			(xy 130.81 30.48) (xy 147.32 30.48)
+		)
+		(stroke
+			(width 0)
+			(type default)
+		)
+	)
+	(wire
+		(pts
 			(xy 34.29 50.8) (xy 36.83 50.8)
 		)
@@
 	(wire
 		(pts
-			(xy 179.07 48.26) (xy 180.34 48.26)
-		)
-		(stroke
-			(width 0)
-			(type default)
-		)
-	)
-	(wire
-		(pts
 			(xy 104.14 50.8) (xy 106.68 50.8)
 		)
@@
 	(wire
 		(pts
+			(xy 180.34 30.48) (xy 180.34 45.72)
+		)
+		(stroke
+			(width 0)
+			(type default)
+		)
+	)
+	(wire
+		(pts
 			(xy 36.83 59.69) (xy 59.69 59.69)
 		)
@@
 	(wire
 		(pts
-			(xy 93.98 15.24) (xy 93.98 30.48)
+			(xy 93.98 21.59) (xy 93.98 30.48)
 		)
 		(stroke
@@
 	(wire
 		(pts
+			(xy 130.81 45.72) (xy 130.81 30.48)
+		)
+		(stroke
+			(width 0)
+			(type default)
+		)
+	)
+	(wire
+		(pts
 			(xy 165.1 72.39) (xy 167.64 72.39)
 		)
@@
 	(wire
 		(pts
+			(xy 128.27 45.72) (xy 130.81 45.72)
+		)
+		(stroke
+			(width 0)
+			(type default)
+		)
+	)
+	(wire
+		(pts
 			(xy 82.55 93.98) (xy 82.55 95.25)
 		)
@@
 	(wire
 		(pts
-			(xy 132.08 33.02) (xy 179.07 33.02)
-		)
-		(stroke
-			(width 0)
-			(type default)
-		)
-	)
-	(wire
-		(pts
 			(xy 129.54 69.85) (xy 132.08 69.85)
 		)
@@
 	(wire
 		(pts
-			(xy 179.07 33.02) (xy 179.07 48.26)
-		)
-		(stroke
-			(width 0)
-			(type default)
-		)
-	)
-	(wire
-		(pts
 			(xy 106.68 50.8) (xy 106.68 52.07)
 		)
@@
 	(wire
 		(pts
-			(xy 179.07 57.15) (xy 179.07 48.26)
-		)
-		(stroke
-			(width 0)
-			(type default)
-		)
-	)
-	(wire
-		(pts
 			(xy 21.59 102.87) (xy 36.83 102.87)
 		)
@@
 	(wire
 		(pts
-			(xy 132.08 45.72) (xy 132.08 33.02)
-		)
-		(stroke
-			(width 0)
-			(type default)
-		)
-	)
-	(wire
-		(pts
 			(xy 165.1 57.15) (xy 166.37 57.15)
 		)
@@
 	(wire
 		(pts
+			(xy 130.81 45.72) (xy 132.08 45.72)
+		)
+		(stroke
+			(width 0)
+			(type default)
+		)
+	)
+	(wire
+		(pts
 			(xy 80.01 50.8) (xy 82.55 50.8)
 		)
@@
 	(wire
 		(pts
+			(xy 149.86 30.48) (xy 180.34 30.48)
+		)
+		(stroke
+			(width 0)
+			(type default)
+		)
+	)
+	(wire
+		(pts
 			(xy 69.85 50.8) (xy 69.85 72.39)
 		)
@@
 		)
 	)
+	(global_label "GND"
+		(shape input)
+		(at 128.27 45.72 180)
+		(fields_autoplaced yes)
+		(effects
+			(font
+				(size 1.27 1.27)
+			)
+			(justify right)
+		)
+		(property "Intersheetrefs" "${INTERSHEET_REFS}"
+			(at 121.4143 45.72 0)
+			(effects
+				(font
+					(size 1.27 1.27)
+				)
+				(justify right)
+				(hide yes)
+			)
+		)
+	)
 	(global_label "ROW3"
 		(shape input)
@@
 		(property "Intersheetrefs" "${INTERSHEET_REFS}"
 			(at 24.13 13.7667 90)
+			(effects
+				(font
+					(size 1.27 1.27)
+				)
+				(justify left)
+				(hide yes)
+			)
+		)
+	)
+	(global_label "GND"
+		(shape input)
+		(at 179.07 57.15 0)
+		(fields_autoplaced yes)
+		(effects
+			(font
+				(size 1.27 1.27)
+			)
+			(justify left)
+		)
+		(property "Intersheetrefs" "${INTERSHEET_REFS}"
+			(at 185.9257 57.15 0)
 			(effects
 				(font
@@
 	(symbol
 		(lib_id "Connector:Conn_01x02_Pin")
-		(at 185.42 48.26 180)
+		(at 149.86 25.4 270)
 		(unit 1)
 		(exclude_from_sim no)
@@
 		(fields_autoplaced yes)
 		(property "Reference" "J1"
-			(at 186.69 45.7199 0)
-			(effects
-				(font
-					(size 1.27 1.27)
-				)
-				(justify right)
+			(at 151.13 24.7649 90)
+			(effects
+				(font
+					(size 1.27 1.27)
+				)
+				(justify left)
 			)
 		)
 		(property "Value" "Conn_01x02_Pin"
-			(at 186.69 48.2599 0)
-			(effects
-				(font
-					(size 1.27 1.27)
-				)
-				(justify right)
+			(at 151.13 27.3049 90)
+			(effects
+				(font
+					(size 1.27 1.27)
+				)
+				(justify left)
 			)
 		)
 		(property "Footprint" "Connector_PinHeader_2.54mm:PinHeader_1x02_P2.54mm_Vertical"
-			(at 185.42 48.26 0)
+			(at 149.86 25.4 0)
 			(effects
 				(font
@@
 		)
 		(property "Datasheet" "~"
-			(at 185.42 48.26 0)
+			(at 149.86 25.4 0)
 			(effects
 				(font
@@
 		)
 		(property "Description" ""
-			(at 185.42 48.26 0)
-			(effects
-				(font
+			(at 149.86 25.4 0)
+			(effects
+				(font
